Commit message: pr2_description: added ft sensor to xacro

File: pr2_description/robots/pr2.urdf.xacro (robot description, xacro)
@@ -12,4 +12,5 @@
   <xacro:include filename="$(find pr2_description)/urdf/upper_arm_v0/upper_arm.urdf.xacro" />
   <xacro:include filename="$(find pr2_description)/urdf/forearm_v0/forearm.urdf.xacro" />
+  <xacro:include filename="$(find pr2_description)/urdf/ft_forearm/pr2_ft_forearm.urdf.xacro" />
   <!-- PR2 gripper -->
   <xacro:include filename="$(find pr2_description)/urdf/gripper_v0/gripper.urdf.xacro" />
@@ -70,8 +71,12 @@
   </xacro:pr2_shoulder_v0>
   <xacro:pr2_upper_arm_v0 side="r" reflect="-1" parent="r_upper_arm_roll_link"/>
-  <xacro:pr2_forearm_v0 side="r" reflect="-1" parent="r_forearm_roll_link">
+  <!--xacro:pr2_forearm_v0 side="r" reflect="-1" parent="r_forearm_roll_link">
     <origin xyz="0 0 0" rpy="0 0 0" />
-  </xacro:pr2_forearm_v0>
-  <xacro:pr2_gripper_v0 reflect="-1.0" side="r" parent="r_wrist_roll_link"
+  </xacro:pr2_forearm_v0-->
+  <xacro:pr2_ft_forearm side="r" reflect="-1" parent="r_forearm_roll_link">
+    <origin xyz="0 0 0" rpy="0 0 0" />
+  </xacro:pr2_ft_forearm>
+  <!--xacro:pr2_gripper_v0 reflect="-1.0" side="r" parent="r_wrist_roll_link" -->
+  <xacro:pr2_gripper_v0 reflect="-1.0" side="r" parent="r_force_torque_link"
                screw_reduction="${4.0/1000.0}"
                gear_ratio="${(729.0/25.0)*(22.0/16.0)}"
@@ -84,5 +89,6 @@
                b="${43.3849/1000.0}"
                r="${91.5/1000.0}" >
-    <origin xyz="0 0 0" rpy="0 0 0" />
+    <!--origin xyz="0 0 0" rpy="0 0 0" /-->
+    <origin xyz="0 0 0" rpy="0 1.5707963267948966 -1.2217304763960306" />
   </xacro:pr2_gripper_v0>
   <xacro:pr2_shoulder_v0 side="l" reflect="1" parent="torso_lift_link">
